Commit message: virtual code

File: turtlebot3_manipulation_description/urdf/turtlebot3_waffle_pi.urdf.xacro (robot description, xacro)
@@ -173,10 +173,4 @@
   </joint>
   <link name="${prefix}camera_link">
-    <collision>
-      <origin xyz="0.005 0.011 0.013" rpy="0 0 0"/>
-      <geometry>
-        <box size="0.015 0.030 0.027"/>
-      </geometry>
-    </collision>
   </link>
   <joint name="${prefix}camera_rgb_joint" type="fixed">
